Commit message: Trying to solve TF Exception message

File: project3/kuka_lwr_arm.urdf (robot description, URDF)
Before this commit: robot lwr, 9 links, 8 joints
Links:
- link world_link: mass 50.0 -> None

File: project3/lwr_robot/lwr_defs/robots/kuka_lwr_arm.urdf (robot description, URDF)
Before this commit: robot lwr, 9 links, 8 joints
Links:
- link world_link: mass 50.0 -> None
