Commit message: Fix URDF

File: utils/kuka_lwr/lwr_robot/lwr_defs/robots/kuka_lwr_arm.urdf (robot description, URDF)
Before this commit: robot lwr, 9 links, 8 joints
Links:
- added link world
Joints:
- removed joint world_link_lwr_arm_base_joint
- added joint world_lwr_arm_base_joint: type fixed, parent world_link, child calib_lwr_arm_base_link, origin xyz=0 0 0.2 rpy=0 0 0
- added joint world_to_lwr: type fixed, parent world, child world_link
